Commit message: enhancing urdf file with correct inertia

File: src/frost_robot_arm/urdf/frost_arm.urdf (robot description, URDF)
Before this commit: robot frost, 8 links, 7 joints
Links:
- link link_0: mass ${link_0_mass} -> 3.107
- link link_1: mass ${link_1_mass} -> 3.579
- link link_2: mass ${link_2_mass} -> 1.8
- link link_3: mass ${link_3_mass} -> 1.8
- link link_4: mass ${link_4_mass} -> 1.041
- link link_5: mass ${link_5_mass} -> 0.014
- link link_base: mass ${link_base_mass} -> 3.528

File: src/frost_robot_arm/urdf/frost_arm_inventor.urdf (robot description, URDF)
Before this commit: robot frost, 8 links, 7 joints
Links:
- link link_0: mass ${link_0_mass} -> 3.107; geometry collision mesh filename=package://frost_robot_arm/meshes/axe2.dae; visual mesh filename=package://frost_robot_arm/meshes/axe2.dae
- link link_1: mass ${link_1_mass} -> 3.579; geometry collision mesh filename=package://frost_robot_arm/meshes/axe3.dae; visual mesh filename=package://frost_robot_arm/meshes/axe3.dae
- link link_2: mass ${link_2_mass} -> 1.8; geometry collision mesh filename=package://frost_robot_arm/meshes/axe4.dae; visual mesh filename=package://frost_robot_arm/meshes/axe4.dae
- link link_3: mass ${link_3_mass} -> 1.8
- link link_4: mass ${link_4_mass} -> 1.041
- link link_5: mass ${link_5_mass} -> 0.014
- link link_base: mass ${link_base_mass} -> 3.528; geometry collision mesh filename=package://frost_robot_arm/meshes/axe1.dae; visual mesh filename=package://frost_robot_arm/meshes/axe1.dae

File: src/frost_robot_arm/urdf/frost_arm_inventor.xacro (robot description, xacro)
@@ -7,13 +7,4 @@
     <color rgba="0.8 0 0 1"/>
   </material>
-  <!--xacro:macro name="cube_inertial" params="width height depth mass *origin">
-    <inertial>
-      <mass value="${mass}" />
-      <xacro:insert_block name="origin" />
-      <inertia ixx="${0.0833333 * mass * (height * height + depth * depth)}" ixy="0.0" ixz="0.0"
-        iyy="${0.0833333 * mass * (width * width + depth * depth)}" iyz="0.0"
-        izz="${0.0833333 * mass * (width * width + height * height)}" />
-    </inertial>
-  </xacro:macro-->
   <!-- mass is entered in kg data a referenced from mikes robot arm in inventor -->
   <xacro:property name="link_base_mass" value="3.528" />
@@ -40,22 +31,22 @@
     <visual>
       <geometry>
-	      <box size="0.15 0.15 0.01"/>
-      </geometry>
-      <origin rpy="0 0 0" xyz="0 0 0.005"/>
-      <material name="blue"/>
-    </visual>
-    <collision>
-      <geometry>
-	      <box size="0.15 0.15 0.01"/>
-      </geometry>
-      <material name="red"/>
-      <origin rpy="0 0 0" xyz="0 0 0.0025"/>
-    </collision>
-    <inertial>
-    <!-- inventor gaves the inertia of a subassambly centerpoint in kg*mm^2-->
-    <mass value="${link_base_mass}"/>
-    <inertia ixx="12943.301" ixy="920.962"   ixz="2494.072"
-                             iyy="34752.194" iyz="-1338.493"
-                                             izz="27487.656"/>
+	      <mesh filename="package://frost_robot_arm/meshes/axe1.dae"/>
+      </geometry>
+      <origin rpy="4.712388981 0 0" xyz="0 0 0.005"/>
+      <material name="blue"/>
+    </visual>
+    <collision>
+      <geometry>
+	      <mesh filename="package://frost_robot_arm/meshes/axe1.dae"/>
+      </geometry>
+      <material name="red"/>
+      <origin rpy="4.712388981 0 0" xyz="0 0 0.0025"/>
+    </collision>
+    <inertial>
+    <!-- inventor gaves the inertia of a subassambly centerpoint in kg*mm^2-->
+      <mass value="${link_base_mass}"/>
+      <inertia ixx="12943.301" ixy="920.962"   ixz="2494.072"
+                               iyy="34752.194" iyz="-1338.493"
+                                               izz="27487.656"/>
     </inertial>
   </link>
@@ -63,15 +54,15 @@
     <visual>
       <geometry>
-	      <box size="0.1 0.1 0.1"/>
-      </geometry>
-      <origin rpy="0 0 0" xyz="0 0 0.05"/>
-      <material name="blue"/>
-    </visual>
-    <collision>
-      <geometry>
-	      <box size="0.1 0.1 0.1"/>
-      </geometry>
-      <material name="red"/>
-      <origin rpy="0 0 0" xyz="0 0 0.05"/>
+	      <mesh filename="package://frost_robot_arm/meshes/axe2.dae"/>
+      </geometry>
+      <origin rpy="0 0 0" xyz="0.052 -0.5615 -0.07"/>
+      <material name="blue"/>
+    </visual>
+    <collision>
+      <geometry>
+	      <mesh filename="package://frost_robot_arm/meshes/axe2.dae"/>
+      </geometry>
+      <material name="red"/>
+      <origin rpy="0 0 0" xyz="0.052 -0.5615 -0.07"/>
     </collision>
     <inertial>
@@ -96,15 +87,15 @@
     <visual>
       <geometry>
-	      <box size="0.1 0.1 0.43"/>
-      </geometry>
-      <origin rpy="0 0 0" xyz="0 0 0.215"/>
-      <material name="blue"/>
-    </visual>
-    <collision>
-      <geometry>
-	      <box size="0.1 0.1 0.35"/>
-      </geometry>
-      <material name="red"/>
-      <origin rpy="0 0 0" xyz="0 0 0.215"/>
+	      <mesh filename="package://frost_robot_arm/meshes/axe3.dae"/>
+      </geometry>
+      <origin rpy="4.712388981 0 -1.570796327" xyz="-0.0043 -0.019 0.40"/>
+      <material name="blue"/>
+    </visual>
+    <collision>
+      <geometry>
+	      <mesh filename="package://frost_robot_arm/meshes/axe3.dae"/>
+      </geometry>
+      <material name="red"/>
+      <origin rpy="4.712388981 0 1.570796327" xyz="0.0 0.019 0.44"/>
     </collision>
     <inertial>
@@ -115,5 +106,5 @@
                                                 izz="85698.080" />
     </inertial>
-    </link>
+  </link>
   <joint name="joint1" type="revolute">
     <axis xyz="0 1 0"/>
@@ -133,14 +124,14 @@
     <visual>
       <geometry>
-        <box size="0.08 0.08 0.21"/>
-      </geometry>
-      <origin rpy="0 0 0" xyz="0 0 0.105"/>
-      <material name="blue"/>
-    </visual>
-    <collision>
-      <geometry>
-        <box size="0.08 0.08 0.21"/>
-      </geometry>
-      <origin rpy="0 0 0" xyz="0 0 0.105"/>
+	      <mesh filename="package://frost_robot_arm/meshes/axe4.dae"/>
+      </geometry>
+      <origin rpy="0 0 3.141592654" xyz="-0.02 0.02 0.255"/>
+      <material name="blue"/>
+    </visual>
+    <collision>
+      <geometry>
+	      <mesh filename="package://frost_robot_arm/meshes/axe4.dae"/>
+      </geometry>
+      <origin rpy="0 0 0" xyz="0 0 0.255"/>
       <material name="red"/>
     </collision>

Commit message: try to get ikfast installed

File: src/frost_robot_arm/urdf/frost_arm.urdf (robot description, URDF)
Before this commit: robot frost, 8 links, 7 joints
Links:
- removed link world
Joints:
- removed joint world_joint
- joint joint0: limit lower=-3.141592654 upper=3.141592654 effort=87 velocity=20 -> lower=-3.141592654 upper=3.141592654 effort=31 velocity=58
- joint joint1: axis 0 1 0 -> -1 0 0; limit lower=-1.570796327 upper=1.570796327 effort=314 velocity=41 -> lower=-1.570796327 upper=1.570796327 effort=472 velocity=41
- joint joint2: axis 0 1 0 -> -1 0 0; limit lower=-2.268928027593 upper=2.617993877991 effort=143 velocity=72 -> lower=-2.268928027593 upper=2.617993877991 effort=109 velocity=72
- joint joint3: limit lower=-2.705260340591 upper=2.705260340591 effort=54 velocity=60 -> lower=-2.705260340591 upper=2.705260340591 effort=91 velocity=60
- joint joint4: axis 0 1 0 -> -1 0 0; limit lower=-1.570796326795 upper=1.570796326795 effort=87 velocity=113 -> lower=-1.570796326795 upper=1.570796326795 effort=109 velocity=113

File: src/frost_robot_arm/urdf/frost_arm.xacro (robot description, xacro)
@@ -3,7 +3,4 @@
   <material name="blue">
     <color rgba="0 0 0.8 0.7"/>
-  </material>
-  <material name="red">
-    <color rgba="0.8 0 0 1"/>
   </material>
   <!--xacro:macro name="cube_inertial" params="width height depth mass *origin">
@@ -24,5 +21,4 @@
   <xacro:property name="link_4_mass" value="1.041" />
   <xacro:property name="link_5_mass" value="0.014" />
-  <link name="world" />
   <!--xacro:unless value="${not connected_to}">
     <joint name="${arm_id}_joint_${connected_to}" type="fixed">
@@ -32,9 +28,4 @@
     </joint>
   </xacro:unless-->
-  <joint name="world_joint" type="fixed">
-    <parent link= "world" />
-    <child link= "link_base" />
-    <origin xyz="0.0 0.0 0.0" rpy="0.0 0.0 0.0" />
-  </joint>
   <link name="link_base">
     <visual>

Commit message: created ikFast algorithem and it works with the robotarm

File: src/frost_robot_arm/urdf/frost_arm.urdf (robot description, URDF)
Before this commit: robot frost, 7 links, 6 joints
Links:
- added link world
Joints:
- added joint world_joint: type fixed, parent world, child link_base, origin xyz=0.0 0.0 0.0 rpy=0.0 0.0 0.0

File: src/frost_robot_arm/urdf/frost_arm.xacro (robot description, xacro)
@@ -3,4 +3,7 @@
   <material name="blue">
     <color rgba="0 0 0.8 0.7"/>
+  </material>
+  <material name="red">
+    <color rgba="0.8 0 0 1"/>
   </material>
   <!--xacro:macro name="cube_inertial" params="width height depth mass *origin">
@@ -21,4 +24,5 @@
   <xacro:property name="link_4_mass" value="1.041" />
   <xacro:property name="link_5_mass" value="0.014" />
+  <link name="world" />
   <!--xacro:unless value="${not connected_to}">
     <joint name="${arm_id}_joint_${connected_to}" type="fixed">
@@ -28,4 +32,9 @@
     </joint>
   </xacro:unless-->
+  <joint name="world_joint" type="fixed">
+    <parent link= "world" />
+    <child link= "link_base" />
+    <origin xyz="0.0 0.0 0.0" rpy="0.0 0.0 0.0" />
+  </joint>
   <link name="link_base">
     <visual>
