Commit message: changes on the urdf files

File: src/frost_robot_arm/urdf/frost_arm.xacro (robot description, xacro)
@@ -16,11 +16,12 @@
     </inertial>
   </xacro:macro>
-  <xacro:property name="link_base_mass" value="0.500" />
-  <xacro:property name="link_0_mass" value="2.515" />
-  <xacro:property name="link_1_mass" value="5.214" />
-  <xacro:property name="link_2_mass" value="2.581" />
-  <xacro:property name="link_3_mass" value="2.581" />
-  <xacro:property name="link_4_mass" value="1.643" />
-  <xacro:property name="link_5_mass" value="0.200" />
+  <!-- mass is entered in kg -->
+  <xacro:property name="link_base_mass" value="3.528" />
+  <xacro:property name="link_0_mass" value="3.107" />
+  <xacro:property name="link_1_mass" value="3.579" />
+  <xacro:property name="link_2_mass" value="1.800" />
+  <xacro:property name="link_3_mass" value="1.800" />
+  <xacro:property name="link_4_mass" value="1.041" />
+  <xacro:property name="link_5_mass" value="0.014" />
   <link name="world" />
   <!--xacro:unless value="${not connected_to}">

Commit message: fixing urdf pyhsikal properties

File: src/frost_robot_arm/urdf/frost_arm.xacro (robot description, xacro)
@@ -91,5 +91,9 @@
     the source to this fact:https://wiki.ros.org/pr2_controller_manager/safety_limits -->
     <!-- this values for effort and velocity are entert without reference. This are only assumptipons-->
-    <limit effort="87" lower="-3.141592654" upper="3.141592654" velocity="20"/>
+    <!-- the planet gear has a ratio of 15,3:1 multipled with the realtion of the cogwheel of the 54 teeth and 24 teeth
+     it multiples up to 15.3 * 54/24 = 34.425. This creates a ration of 34.425:1-->
+    <!-- form datasheet permited repeatable peak torque 176Nm-->
+    <!-- with a ratio of 34.425 and a maximal motor speed of 2000 rad/min, we get a maximal output speed of 58 rad/min-->
+    <limit effort="87" lower="-3.141592654" upper="3.141592654" velocity="58"/>
   </joint>
   <link name="link_1">
@@ -117,5 +121,5 @@
     </link>
   <joint name="joint1" type="revolute">
-    <axis xyz="0 1 0"/>
+    <axis xyz="-1 0 0"/>
     <parent link="link_0"/>
     <child link="link_1"/>
@@ -125,8 +129,7 @@
     <!-- effort for the harmonic drive is given in Nm and velocity in rotation per minit-->
     <!--effort specification for the HFUC-25-160-2UH: https://harmonicdrive.de/fileadmin/user_upload/2014_12_ED_1019644_HFUC_2UH.pdf -->
-    <!-- due to data sheet by a ratio of 160 and a Maximum input speed 7500 (oil lubrication) you can get up to 46.875 output rotation
-         so to be carfule we use the mean value between Maximum input speed 5600 (oil lubrication) and Maximum input speed (grease lubrication)
-         which is 40.9375 roundet to 41 rotation per minit maximum velocity-->
-    <limit effort="314" lower="-1.570796327" upper="1.570796327" velocity="41"/>
+    <!-- form datasheet permited repeatable peak torque 176Nm-->
+    <!-- with a ratio of 160 and a maximal motor speed of XXX rad/min, we get a maximal output speed of XXX rad/min-->
+    <limit effort="176" lower="-1.570796327" upper="1.570796327" velocity="41"/>
   </joint>
   <link name="link_2">
@@ -154,16 +157,15 @@
   </link>
   <joint name="joint2" type="revolute">
-    <origin rpy="0 0 0" xyz="0 0 0.43"/>
+    <axis xyz="-1 0 0"/>
     <parent link="link_1"/>
     <child link="link_2"/>
-    <axis xyz="0 1 0"/>
+    <origin rpy="0 0 0" xyz="0 0 0.43"/>
     <!-- effort is for revolut joints in Nm for translatoric joints N
     the source to this fact:https://wiki.ros.org/pr2_controller_manager/safety_limits -->
     <!-- effort for the harmonic drive is given in Nm and velocity in rotation per minit-->
     <!--effort specification for the CSG-17-120-2UH: https://harmonicdrive.de/fileadmin/user_upload/2014_12_ED_1019642_CSG_2UH.pdf -->
-    <!-- due to data sheet by a ratio is 120 and a Maximum input speed 10000 (oil lubrication) you can get up to 83.3333 output rotation
-         so to be carfule we use the mean value between Maximum input speed 7300 (oil lubrication) and Maximum input speed (grease lubrication)
-         which is 72.0832 roundet to 72 rotation per minit maximum velocity-->
-    <limit effort="143" lower="-2.268928027593" upper="2.617993877991" velocity="72"/>
+    <!-- form datasheet permited repeatable peak torque 176Nm-->
+    <!-- with a ratio of 120 and a maximal motor speed of XXX rad/min, we get a maximal output speed of XXX rad/min-->
+    <limit effort="70" lower="-2.268928027593" upper="2.617993877991" velocity="72"/>
   </joint>
   <link name="link_3">
@@ -191,16 +193,15 @@
   </link>
   <joint name="joint3" type="revolute">
-    <origin rpy="0 0 0" xyz="0.0 0.0 0.21"/>
+    <axis xyz="0 0 1"/>
     <parent link="link_2"/>
     <child link="link_3"/>
-    <axis xyz="0 0 1"/>
+    <origin rpy="0 0 0" xyz="0.0 0.0 0.21"/>
     <!-- effort is for revolut joints in Nm for translatoric joints N
     the source to this fact:https://wiki.ros.org/pr2_controller_manager/safety_limits -->
     <!-- effort for the harmonic drive is given in Nm and velocity in rotation per minit-->
     <!--effort specification for the CSF-14-100-2XH : https://harmonicdrive.de/fileadmin/user_upload/2014_12_ED_1019649_CSF_Mini.pdf -->
-    <!-- due to data sheet by a ratio is 100 and a Maximum input speed 8500 (oil lubrication) you can get up to 85 output rotation
-         so to be carfule we use the mean value between Maximum input speed 3500 (oil lubrication) and Maximum input speed (grease lubrication)
-         which is 60-->
-    <limit effort="54" lower="-2.705260340591" upper="2.705260340591" velocity="60"/>
+    <!-- form datasheet permited repeatable peak torque 28Nm-->
+    <!-- with a ratio of 100 and a maximal motor speed of XXX rad/min, we get a maximal output speed of XXX rad/min-->
+    <limit effort="28" lower="-2.705260340591" upper="2.705260340591" velocity="60"/>
   </joint>
   <link name="link_4">
@@ -228,16 +229,15 @@
   </link>
   <joint name="joint4" type="revolute">
-    <origin rpy="0 0 0" xyz="0 0.0 0.21"/>
+    <axis xyz="-1 0 0"/>
     <parent link="link_3"/>
     <child link="link_4"/>
-    <axis xyz="0 1 0"/>
+    <origin rpy="0 0 0" xyz="0 0.0 0.21"/>
     <!-- effort is for revolut joints in Nm for translatoric joints N
     the source to this fact:https://wiki.ros.org/pr2_controller_manager/safety_limits -->
     <!-- effort for the harmonic drive is given in Nm and velocity in rotation per minit -->
-    <!--effort specification for the HFUC-14-100-2UH : https://harmonicdrive.de/fileadmin/user_upload/2014_12_ED_1019644_HFUC_2UH.pdf -->
-    <!-- due to data sheet by a ratio is 100 and a Maximum input speed 14000 (oil lubrication) you can get up to 140 output rotation
-         so to be carfule we use the mean value between Maximum input speed 8500 (oil lubrication) and Maximum input speed (grease lubrication)
-         which is 112.5 roundet to 113 rotation per minit maximum velocity-->
-    <limit effort="87" lower="-1.570796326795" upper="1.570796326795" velocity="113"/>
+    <!--effort specification for the CSG-17-120-2UH: https://harmonicdrive.de/fileadmin/user_upload/2014_12_ED_1019642_CSG_2UH.pdf -->
+    <!-- form datasheet permited repeatable peak torque 70Nm-->
+    <!-- with a ratio of 120 and a maximal motor speed of XXX rad/min, we get a maximal output speed of XXX rad/min-->
+    <limit effort="70" lower="-1.570796326795" upper="1.570796326795" velocity="113"/>
   </joint>
   <link name="link_5">
@@ -265,8 +265,8 @@
   </link>
   <joint name="joint5" type="revolute">
-    <origin rpy="0 0 0" xyz="0 0 0.125"/>
+    <axis xyz="0 0 1"/>
     <parent link="link_4"/>
     <child link="link_5"/>
-    <axis xyz="0 0 1"/>
+    <origin rpy="0 0 0" xyz="0 0 0.125"/>
     <!-- effort is for revolut joints in Nm for translatoric joints N
     the source to this fact:https://wiki.ros.org/pr2_controller_manager/safety_limits -->

Commit message: update urdf file correct Rotation Moment in Nm

File: src/frost_robot_arm/urdf/frost_arm.xacro (robot description, xacro)
@@ -95,5 +95,5 @@
     <!-- form datasheet permited repeatable peak torque 176Nm-->
     <!-- with a ratio of 34.425 and a maximal motor speed of 2000 rad/min, we get a maximal output speed of 58 rad/min-->
-    <limit effort="87" lower="-3.141592654" upper="3.141592654" velocity="58"/>
+    <limit effort="31" lower="-3.141592654" upper="3.141592654" velocity="58"/>
   </joint>
   <link name="link_1">
@@ -131,5 +131,5 @@
     <!-- form datasheet permited repeatable peak torque 176Nm-->
     <!-- with a ratio of 160 and a maximal motor speed of XXX rad/min, we get a maximal output speed of XXX rad/min-->
-    <limit effort="176" lower="-1.570796327" upper="1.570796327" velocity="41"/>
+    <limit effort="472" lower="-1.570796327" upper="1.570796327" velocity="41"/>
   </joint>
   <link name="link_2">
@@ -167,5 +167,5 @@
     <!-- form datasheet permited repeatable peak torque 176Nm-->
     <!-- with a ratio of 120 and a maximal motor speed of XXX rad/min, we get a maximal output speed of XXX rad/min-->
-    <limit effort="70" lower="-2.268928027593" upper="2.617993877991" velocity="72"/>
+    <limit effort="109" lower="-2.268928027593" upper="2.617993877991" velocity="72"/>
   </joint>
   <link name="link_3">
@@ -203,5 +203,5 @@
     <!-- form datasheet permited repeatable peak torque 28Nm-->
     <!-- with a ratio of 100 and a maximal motor speed of XXX rad/min, we get a maximal output speed of XXX rad/min-->
-    <limit effort="28" lower="-2.705260340591" upper="2.705260340591" velocity="60"/>
+    <limit effort="91" lower="-2.705260340591" upper="2.705260340591" velocity="60"/>
   </joint>
   <link name="link_4">
@@ -239,5 +239,5 @@
     <!-- form datasheet permited repeatable peak torque 70Nm-->
     <!-- with a ratio of 120 and a maximal motor speed of XXX rad/min, we get a maximal output speed of XXX rad/min-->
-    <limit effort="70" lower="-1.570796326795" upper="1.570796326795" velocity="113"/>
+    <limit effort="109" lower="-1.570796326795" upper="1.570796326795" velocity="113"/>
   </joint>
   <link name="link_5">

Commit message: anpassen des kommentarbereichs. muss noch effort und velocity anpassen

File: src/frost_robot_arm/urdf/frost_arm.xacro (robot description, xacro)
@@ -88,10 +88,12 @@
     <parent link="link_base"/>
     <child link="link_0"/>
-    <!-- effort is for revolut joints in Nm for translatoric joints N
+    <!-- effort is for revolut joints in Nm for translatoric joints N and the velocity is in rad/s
     the source to this fact:https://wiki.ros.org/pr2_controller_manager/safety_limits -->
     <!-- this values for effort and velocity are entert without reference. This are only assumptipons-->
     <!-- the planet gear has a ratio of 15,3:1 multipled with the realtion of the cogwheel of the 54 teeth and 24 teeth
      it multiples up to 15.3 * 54/24 = 34.425. This creates a ration of 34.425:1-->
-    <!-- form datasheet permited repeatable peak torque 176Nm-->
+    <!-- The actuator what we are using is the steppermotor 23HS22-2804S-PG15 with a maximum rotation per minit of 400 n/min
+    and a maximum Moment of 0,916 Nm-->
+    <!-- also a two gears a used with a ratio of 54 to 24 thats a ratio of 2,25-->
     <!-- with a ratio of 34.425 and a maximal motor speed of 2000 rad/min, we get a maximal output speed of 58 rad/min-->
     <limit effort="31" lower="-3.141592654" upper="3.141592654" velocity="58"/>
@@ -125,10 +127,12 @@
     <child link="link_1"/>
     <origin rpy="0 0 0" xyz="0 0 0.1"/>
-    <!-- effort is for revolut joints in Nm for translatoric joints N
+    <!-- effort is for revolut joints in Nm for translatoric joints N and the velocity is in rad/s
     the source to this fact:https://wiki.ros.org/pr2_controller_manager/safety_limits -->
     <!-- effort for the harmonic drive is given in Nm and velocity in rotation per minit-->
     <!--effort specification for the HFUC-25-160-2UH: https://harmonicdrive.de/fileadmin/user_upload/2014_12_ED_1019644_HFUC_2UH.pdf -->
     <!-- form datasheet permited repeatable peak torque 176Nm-->
-    <!-- with a ratio of 160 and a maximal motor speed of XXX rad/min, we get a maximal output speed of XXX rad/min-->
+    <!-- The actuator what we are using is the steppermotor ST8918S4508-A with a maximum rotation per minit of 150 n/min
+    and a maximum Moment of 2,95 Nm-->
+    <!-- with a ratio of 160 and a maximal motor speed of 150 rad/min, we get a maximal output speed of 0,0156 rad/min-->
     <limit effort="472" lower="-1.570796327" upper="1.570796327" velocity="41"/>
   </joint>
@@ -161,10 +165,12 @@
     <child link="link_2"/>
     <origin rpy="0 0 0" xyz="0 0 0.43"/>
-    <!-- effort is for revolut joints in Nm for translatoric joints N
+    <!-- effort is for revolut joints in Nm for translatoric joints N and the velocity is in rad/s
     the source to this fact:https://wiki.ros.org/pr2_controller_manager/safety_limits -->
     <!-- effort for the harmonic drive is given in Nm and velocity in rotation per minit-->
     <!--effort specification for the CSG-17-120-2UH: https://harmonicdrive.de/fileadmin/user_upload/2014_12_ED_1019642_CSG_2UH.pdf -->
     <!-- form datasheet permited repeatable peak torque 176Nm-->
-    <!-- with a ratio of 120 and a maximal motor speed of XXX rad/min, we get a maximal output speed of XXX rad/min-->
+    <!-- The actuator what we are using is the steppermotor ST6018X3008-A with a maximum rotation per minit of 400 n/min
+    and a maximum Moment of 0,916 Nm-->
+    <!-- with a ratio of 120 and a maximal motor speed of 400 rad/min, we get a maximal output speed of 0,075 rad/s-->
     <limit effort="109" lower="-2.268928027593" upper="2.617993877991" velocity="72"/>
   </joint>
@@ -197,11 +203,13 @@
     <child link="link_3"/>
     <origin rpy="0 0 0" xyz="0.0 0.0 0.21"/>
-    <!-- effort is for revolut joints in Nm for translatoric joints N
+    <!-- effort is for revolut joints in Nm for translatoric joints N and the velocity is in rad/s
     the source to this fact:https://wiki.ros.org/pr2_controller_manager/safety_limits -->
     <!-- effort for the harmonic drive is given in Nm and velocity in rotation per minit-->
     <!--effort specification for the CSF-14-100-2XH : https://harmonicdrive.de/fileadmin/user_upload/2014_12_ED_1019649_CSF_Mini.pdf -->
     <!-- form datasheet permited repeatable peak torque 28Nm-->
-    <!-- with a ratio of 100 and a maximal motor speed of XXX rad/min, we get a maximal output speed of XXX rad/min-->
-    <limit effort="91" lower="-2.705260340591" upper="2.705260340591" velocity="60"/>
+    <!-- The actuator what we are using is the steppermotor ST4118L3004-B with a maximum rotation per minit of 450 n/min
+    and a maximum Moment of 0,531 Nm-->
+    <!-- with a ratio of 100 and a maximal motor speed of 450 rad/min, we get a maximal output speed of 0,0555 rad/s-->
+    <limit effort="53" lower="-2.705260340591" upper="2.705260340591" velocity="60"/>
   </joint>
   <link name="link_4">
@@ -233,9 +241,11 @@
     <child link="link_4"/>
     <origin rpy="0 0 0" xyz="0 0.0 0.21"/>
-    <!-- effort is for revolut joints in Nm for translatoric joints N
+    <!-- effort is for revolut joints in Nm for translatoric joints N and the velocity is in rad/s
     the source to this fact:https://wiki.ros.org/pr2_controller_manager/safety_limits -->
     <!-- effort for the harmonic drive is given in Nm and velocity in rotation per minit -->
     <!--effort specification for the CSG-17-120-2UH: https://harmonicdrive.de/fileadmin/user_upload/2014_12_ED_1019642_CSG_2UH.pdf -->
     <!-- form datasheet permited repeatable peak torque 70Nm-->
+    <!-- The actuator what we are using is the steppermotor ST6018X3008-A with a maximum rotation per minit of 400 n/min
+    and a maximum Moment of 0,916 Nm-->
     <!-- with a ratio of 120 and a maximal motor speed of XXX rad/min, we get a maximal output speed of XXX rad/min-->
     <limit effort="109" lower="-1.570796326795" upper="1.570796326795" velocity="113"/>
@@ -269,7 +279,9 @@
     <child link="link_5"/>
     <origin rpy="0 0 0" xyz="0 0 0.125"/>
-    <!-- effort is for revolut joints in Nm for translatoric joints N
+    <!-- effort is for revolut joints in Nm for translatoric joints N and the velocity is in rad/s
     the source to this fact:https://wiki.ros.org/pr2_controller_manager/safety_limits -->
     <!-- this values for effort and velocity are entert without reference. This are only assumptipons-->
+    <!-- The actuator what we are using is the steppermotor ST6018X3008-A with a maximum rotation per minit of 400 n/min
+    and a maximum Moment of 0,916 Nm-->
     <limit effort="2" lower="-3.14159265359" upper="3.14159265359" velocity="10"/>
   </joint>
