Commit message: final version of real arm

File: src/frost_robot_arm/urdf/frost_arm.xacro (robot description, xacro)
@@ -88,12 +88,13 @@
     <parent link="link_base"/>
     <child link="link_0"/>
-    <!-- effort is for revolut joints in Nm for translatoric joints N
+    <!-- effort is for revolut joints in Nm for translatoric joints N, velocity is rad/sec
     the source to this fact:https://wiki.ros.org/pr2_controller_manager/safety_limits -->
     <!-- this values for effort and velocity are entert without reference. This are only assumptipons-->
+    <!-- specification of the motor-gear 23HS22-2804S-PG15-->
     <!-- the planet gear has a ratio of 15,3:1 multipled with the realtion of the cogwheel of the 54 teeth and 24 teeth
      it multiples up to 15.3 * 54/24 = 34.425. This creates a ration of 34.425:1-->
-    <!-- form datasheet permited repeatable peak torque 176Nm-->
-    <!-- with a ratio of 34.425 and a maximal motor speed of 2000 rad/min, we get a maximal output speed of 58 rad/min-->
-    <limit effort="31" lower="-3.141592654" upper="3.141592654" velocity="58"/>
+    <!-- form datasheet permited repeatable peak torque 11.06Nm we use 8.5 Nm and multiply it with 54/24 and get 19.125-->
+    <!-- with a ratio of 34.425 and a maximal motor speed of 344,25 n/min, we get a maximal output speed of 1,048 rad/s-->
+    <limit effort="19" lower="-3.141592654" upper="3.141592654" velocity="1.048"/>
   </joint>
   <link name="link_1">
@@ -125,11 +126,12 @@
     <child link="link_1"/>
     <origin rpy="0 0 0" xyz="0 0 0.1"/>
-    <!-- effort is for revolut joints in Nm for translatoric joints N
+    <!-- effort is for revolut joints in Nm for translatoric joints N, velocity is rad/sec
     the source to this fact:https://wiki.ros.org/pr2_controller_manager/safety_limits -->
     <!-- effort for the harmonic drive is given in Nm and velocity in rotation per minit-->
     <!--effort specification for the HFUC-25-160-2UH: https://harmonicdrive.de/fileadmin/user_upload/2014_12_ED_1019644_HFUC_2UH.pdf -->
-    <!-- form datasheet permited repeatable peak torque 176Nm-->
-    <!-- with a ratio of 160 and a maximal motor speed of XXX rad/min, we get a maximal output speed of XXX rad/min-->
-    <limit effort="472" lower="-1.570796327" upper="1.570796327" velocity="41"/>
+    <!-- specification of the motor ST8918S4508-A-->
+    <!-- with a ratio of 160 and a maximal motor speed of 150 n/min, we get a maximal output speed of 0,098 rad/sec.
+    Experiments showed even 0.348 rad/sec are also possible-->
+    <limit effort="236" lower="-1.570796327" upper="1.570796327" velocity="0.348"/>
   </joint>
   <link name="link_2">
@@ -161,11 +163,13 @@
     <child link="link_2"/>
     <origin rpy="0 0 0" xyz="0 0 0.43"/>
-    <!-- effort is for revolut joints in Nm for translatoric joints N
+    <!-- effort is for revolut joints in Nm for translatoric joints N, velocity is rad/sec
     the source to this fact:https://wiki.ros.org/pr2_controller_manager/safety_limits -->
     <!-- effort for the harmonic drive is given in Nm and velocity in rotation per minit-->
-    <!--effort specification for the CSG-17-120-2UH: https://harmonicdrive.de/fileadmin/user_upload/2014_12_ED_1019642_CSG_2UH.pdf -->
+    <!--effort specification for the gear CSG-17-120-2UH: https://harmonicdrive.de/fileadmin/user_upload/2014_12_ED_1019642_CSG_2UH.pdf -->
+    <!-- specification of the motor ST6018X3008-A-->
     <!-- form datasheet permited repeatable peak torque 176Nm-->
-    <!-- with a ratio of 120 and a maximal motor speed of XXX rad/min, we get a maximal output speed of XXX rad/min-->
-    <limit effort="109" lower="-2.268928027593" upper="2.617993877991" velocity="72"/>
+    <!-- with a ratio of 120 and a maximal motor speed of 400 rad/min, we get a maximal output speed of 0,349 rad/sec
+      experiments showed even 0,522 rad/sec are also possible-->
+    <limit effort="109" lower="-2.268928027593" upper="2.617993877991" velocity="0.522"/>
   </joint>
   <link name="link_3">
@@ -200,8 +204,10 @@
     the source to this fact:https://wiki.ros.org/pr2_controller_manager/safety_limits -->
     <!-- effort for the harmonic drive is given in Nm and velocity in rotation per minit-->
-    <!--effort specification for the CSF-14-100-2XH : https://harmonicdrive.de/fileadmin/user_upload/2014_12_ED_1019649_CSF_Mini.pdf -->
+    <!--effort specification for the Gear CSF-14-100-2XH : https://harmonicdrive.de/fileadmin/user_upload/2014_12_ED_1019649_CSF_Mini.pdf -->
+    <!-- specification of the motor ST4118X3004-B-->
     <!-- form datasheet permited repeatable peak torque 28Nm-->
-    <!-- with a ratio of 100 and a maximal motor speed of XXX rad/min, we get a maximal output speed of XXX rad/min-->
-    <limit effort="91" lower="-2.705260340591" upper="2.705260340591" velocity="60"/>
+    <!-- with a ratio of 100 and a maximal motor speed of 450 rad/min, we get a maximal output speed of 0,471 rad/sec
+      we use the doubled velocity, but we coulnd tested thet velocity, because the joint didnt exist-->
+    <limit effort="91" lower="-2.705260340591" upper="2.705260340591" velocity="0.942"/>
   </joint>
   <link name="link_4">
@@ -236,8 +242,10 @@
     the source to this fact:https://wiki.ros.org/pr2_controller_manager/safety_limits -->
     <!-- effort for the harmonic drive is given in Nm and velocity in rotation per minit -->
-    <!--effort specification for the CSG-17-120-2UH: https://harmonicdrive.de/fileadmin/user_upload/2014_12_ED_1019642_CSG_2UH.pdf -->
+    <!--effort specification for the Gear CSG-17-120-2UH: https://harmonicdrive.de/fileadmin/user_upload/2014_12_ED_1019642_CSG_2UH.pdf -->
+    <!-- specification of the motor ST6018X3008-A-->
     <!-- form datasheet permited repeatable peak torque 70Nm-->
-    <!-- with a ratio of 120 and a maximal motor speed of XXX rad/min, we get a maximal output speed of XXX rad/min-->
-    <limit effort="109" lower="-1.570796326795" upper="1.570796326795" velocity="113"/>
+    <!-- with a ratio of 120 and a maximal motor speed of 400 rad/min, we get a maximal output speed of 0,349 rad/sec
+      experimental we showed even 1,256 rad/sec is possible-->
+    <limit effort="109" lower="-1.570796326795" upper="1.570796326795" velocity="1.256"/>
   </joint>
   <link name="link_5">
@@ -272,5 +280,5 @@
     the source to this fact:https://wiki.ros.org/pr2_controller_manager/safety_limits -->
     <!-- this values for effort and velocity are entert without reference. This are only assumptipons-->
-    <limit effort="2" lower="-3.14159265359" upper="3.14159265359" velocity="10"/>
+    <limit effort="100" lower="-3.14159265359" upper="3.14159265359" velocity="1"/>
   </joint>
 </robot>
